File: MAP_input1.sch (KiCad schematic (older format))
At the start: 4 parts, among them U6 MPX4100A

Commit message: DFH mans up a bit. Perhaps usable for something at this point, like making trips to the local store ;)
I connected TA pins to sub circuits, fixed a number if items discussed in the DIYEFI forums. This is it's 21st version, so it was time for it to man up a bit, and become something potentially useful.

Signed-off-by: Jared Harvey <TortiseGIT@jaredharvey.com>
Parts:
- C22: Field10 (none) -> multilayer ceramic; Field11 (none) -> other,more,stuff; Field4 (none) -> newark,97M4164; Field5 (none) -> vendor1, smd w hem; Field6 (none) -> vendor2, thru w hem; Field7 (none) -> vendor2, smd w hem; Field8 (none) -> 50,V; Field9 (none) -> 10,%
- C23: Field10 (none) -> multilayer ceramic; Field11 (none) -> other,more,stuff; Field4 (none) -> newark,75M7682; Field5 (none) -> vendor1, smd w hem; Field6 (none) -> vendor2, thru w hem; Field7 (none) -> vendor2, smd w hem; Field8 (none) -> 50,V; Field9 (none) -> 10,%
- C24: Field10 (none) -> multilayer ceramic; Field11 (none) -> other,more,stuff; Field4 (none) -> newark,19C6191; Field5 (none) -> vendor1, smd w hem; Field6 (none) -> vendor2, thru w hem; Field7 (none) -> vendor2, smd w hem; Field8 (none) -> 100,V; Field9 (none) -> 5,%
- U6: Field10 (none) -> x; Field11 (none) -> other,more,stuff; Field4 (none) -> newark,75C3857; Field5 (none) -> vendor1, smd w hem; Field6 (none) -> vendor2, thru w hem; Field7 (none) -> vendor2, smd w hem; Field8 (none) -> x,x; Field9 (none) -> x,x
Changed lines of the file:
@@
-EESchema Schematic File Version 1
-LIBS:power,./freeEMS_lib,device,conn,linear,regul,74xx,cmos4000,adc-dac,memory,xilinx,special,microcontrollers,dsp,microchip,analog_switches,motorola,texas,intel,audio,interface,digital-audio,philips,display,cypress,siliconi,contrib,valves,./freeEMS_1.cache
-EELAYER 23  0
+EESchema Schematic File Version 2  date 9/10/2011 11:43:50 AM
+LIBS:power
+LIBS:freeEMS_lib
+LIBS:device
+LIBS:conn
+LIBS:linear
+LIBS:regul
+LIBS:74xx
+LIBS:cmos4000
+LIBS:adc-dac
+LIBS:memory
+LIBS:xilinx
+LIBS:special
+LIBS:microcontrollers
+LIBS:dsp
+LIBS:microchip
+LIBS:analog_switches
+LIBS:motorola
+LIBS:texas
+LIBS:intel
+LIBS:audio
+LIBS:interface
+LIBS:digital-audio
+LIBS:philips
+LIBS:display
+LIBS:cypress
+LIBS:siliconi
+LIBS:contrib
+LIBS:valves
+LIBS:freeEMS_1-cache
+EELAYER 25  0
 EELAYER END
 $Descr A 11000 8500
+encoding utf-8
 Sheet 17 41
-Title "freeEMS 1.0"
-Date "15 nov 2008"
-Rev "A.20"
-Comp "diyefi.org"
+Title "DFH for freeEMS"
+Date "10 sep 2011"
+Rev "A.21"
+Comp "FreeEMS.org"
 Comment1 "MAP_input.sch"
 Comment2 ""
@@
 $Comp
 L MPX4100A U6
-U 1 1 48B144B7
+U 1 1 4E6B7072
 P 5100 1500
-F 0 "U6" H 4850 2050 70  0000 C C
-F 1 "MPX4100A" H 5050 950 70  0000 C C
-F 2 "SOP_case_482" V 1130 2600 60  0001 C C
-F 4 "newark,75C3857" V 1130 2600 60  0001 C C
-F 5 "vendor1, smd w hem" V 1130 2600 60  0001 C C
-F 6 "vendor2, thru w hem" V 1130 2600 60  0001 C C
-F 7 "vendor2, smd w hem" V 1130 2600 60  0001 C C
-F 8 "x,x" V 1130 2600 60  0001 C C
-F 9 "x,x" V 1130 2600 60  0001 C C
-F 10 "x" V 1130 2600 60  0001 C C
-F 11 "other,more,stuff" V 1130 2600 60  0001 C C
+F 0 "U6" H 4850 2050 70  0000 C CNN
+F 1 "MPX4100A" H 5050 950 70  0000 C CNN
+F 2 "SOP_case_482" V 1130 2600 60  0001 C CNN
+F 4 "newark,75C3857" V 1130 2600 60  0001 C CNN "Field4"
+F 5 "vendor1, smd w hem" V 1130 2600 60  0001 C CNN "Field5"
+F 6 "vendor2, thru w hem" V 1130 2600 60  0001 C CNN "Field6"
+F 7 "vendor2, smd w hem" V 1130 2600 60  0001 C CNN "Field7"
+F 8 "x,x" V 1130 2600 60  0001 C CNN "Field8"
+F 9 "x,x" V 1130 2600 60  0001 C CNN "Field9"
+F 10 "x" V 1130 2600 60  0001 C CNN "Field10"
+F 11 "other,more,stuff" V 1130 2600 60  0001 C CNN "Field11"
 	1    5100 1500
 	1    0    0    -1
@@
 Wire Wire Line
 	4150 1400 4150 1200
-Text GLabel 2400 1600 0    60   BiDi
+Text HLabel 2400 1600 0    60   BiDi ~ 0
 analog_sensor_gnd
 $Comp
@@
 U 1 1 488D2158
 P 3800 1400
-F 0 "C23" H 3850 1500 50  0000 L C
-F 1 ".01uF" H 3850 1300 50  0000 L C
-F 2 "C1V7" V 1130 2600 60  0001 C C
-F 4 "newark,75M7682" V 1130 2600 60  0001 C C
-F 5 "vendor1, smd w hem" V 1130 2600 60  0001 C C
-F 6 "vendor2, thru w hem" V 1130 2600 60  0001 C C
-F 7 "vendor2, smd w hem" V 1130 2600 60  0001 C C
-F 8 "50,V" V 1130 2600 60  0001 C C
-F 9 "10,%" V 1130 2600 60  0001 C C
-F 10 "multilayer ceramic" V 1130 2600 60  0001 C C
-F 11 "other,more,stuff" V 1130 2600 60  0001 C C
+F 0 "C23" H 3850 1500 50  0000 L CNN
+F 1 ".01uF" H 3850 1300 50  0000 L CNN
+F 2 "C1V7" V 1130 2600 60  0001 C CNN
+F 4 "newark,75M7682" V 1130 2600 60  0001 C CNN "Field4"
+F 5 "vendor1, smd w hem" V 1130 2600 60  0001 C CNN "Field5"
+F 6 "vendor2, thru w hem" V 1130 2600 60  0001 C CNN "Field6"
+F 7 "vendor2, smd w hem" V 1130 2600 60  0001 C CNN "Field7"
+F 8 "50,V" V 1130 2600 60  0001 C CNN "Field8"
+F 9 "10,%" V 1130 2600 60  0001 C CNN "Field9"
+F 10 "multilayer ceramic" V 1130 2600 60  0001 C CNN "Field10"
+F 11 "other,more,stuff" V 1130 2600 60  0001 C CNN "Field11"
 	1    3800 1400
 	1    0    0    -1
@@
 U 1 1 488D2153
 P 3800 1800
-F 0 "C24" H 3850 1900 50  0000 L C
-F 1 "470pF" H 3850 1700 50  0000 L C
-F 2 "C1V7" V 1130 2600 60  0001 C C
-F 4 "newark,19C6191" V 1130 2600 60  0001 C C
-F 5 "vendor1, smd w hem" V 1130 2600 60  0001 C C
-F 6 "vendor2, thru w hem" V 1130 2600 60  0001 C C
-F 7 "vendor2, smd w hem" V 1130 2600 60  0001 C C
-F 8 "100,V" V 1130 2600 60  0001 C C
-F 9 "5,%" V 1130 2600 60  0001 C C
-F 10 "multilayer ceramic" V 1130 2600 60  0001 C C
-F 11 "other,more,stuff" V 1130 2600 60  0001 C C
+F 0 "C24" H 3850 1900 50  0000 L CNN
+F 1 "470pF" H 3850 1700 50  0000 L CNN
+F 2 "C1V7" V 1130 2600 60  0001 C CNN
+F 4 "newark,19C6191" V 1130 2600 60  0001 C CNN "Field4"
+F 5 "vendor1, smd w hem" V 1130 2600 60  0001 C CNN "Field5"
+F 6 "vendor2, thru w hem" V 1130 2600 60  0001 C CNN "Field6"
+F 7 "vendor2, smd w hem" V 1130 2600 60  0001 C CNN "Field7"
+F 8 "100,V" V 1130 2600 60  0001 C CNN "Field8"
+F 9 "5,%" V 1130 2600 60  0001 C CNN "Field9"
+F 10 "multilayer ceramic" V 1130 2600 60  0001 C CNN "Field10"
+F 11 "other,more,stuff" V 1130 2600 60  0001 C CNN "Field11"
 	1    3800 1800
 	1    0    0    -1
@@
 $Comp
 L C C22
-U 1 1 488D2133
+U 1 1 4E6B6FEA
 P 3300 1400
-F 0 "C22" H 3350 1500 50  0000 L C
-F 1 ".1uF" H 3350 1300 50  0000 L C
-F 2 "C1V7" V 1130 2600 60  0001 C C
-F 4 "newark,97M4164" V 1130 2600 60  0001 C C
-F 5 "vendor1, smd w hem" V 1130 2600 60  0001 C C
-F 6 "vendor2, thru w hem" V 1130 2600 60  0001 C C
-F 7 "vendor2, smd w hem" V 1130 2600 60  0001 C C
-F 8 "50,V" V 1130 2600 60  0001 C C
-F 9 "10,%" V 1130 2600 60  0001 C C
-F 10 "multilayer ceramic" V 1130 2600 60  0001 C C
-F 11 "other,more,stuff" V 1130 2600 60  0001 C C
+F 0 "C22" H 3350 1500 50  0000 L CNN
+F 1 ".1uF" H 3350 1300 50  0000 L CNN
+F 2 "C1V7" V 1130 2600 60  0001 C CNN
+F 4 "newark,97M4164" V 1130 2600 60  0001 C CNN "Field4"
+F 5 "vendor1, smd w hem" V 1130 2600 60  0001 C CNN "Field5"
+F 6 "vendor2, thru w hem" V 1130 2600 60  0001 C CNN "Field6"
+F 7 "vendor2, smd w hem" V 1130 2600 60  0001 C CNN "Field7"
+F 8 "50,V" V 1130 2600 60  0001 C CNN "Field8"
+F 9 "10,%" V 1130 2600 60  0001 C CNN "Field9"
+F 10 "multilayer ceramic" V 1130 2600 60  0001 C CNN "Field10"
+F 11 "other,more,stuff" V 1130 2600 60  0001 C CNN "Field11"
 	1    3300 1400
 	1    0    0    -1
 $EndComp
-Text GLabel 2400 1200 0    60   Input
+Text HLabel 2400 1200 0    60   Input ~ 0
 5v reg
-Text GLabel 2400 2000 0    60   Output
+Text HLabel 2400 2000 0    60   Output ~ 0
 analog_sensor_MAP
 $EndSCHEMATC
