File: an_protect2.sch (KiCad schematic (older format))
At the start: 15 parts

Commit message: DFH mans up a bit. Perhaps usable for something at this point, like making trips to the local store ;)
I connected TA pins to sub circuits, fixed a number if items discussed in the DIYEFI forums. This is it's 21st version, so it was time for it to man up a bit, and become something potentially useful.

Signed-off-by: Jared Harvey <TortiseGIT@jaredharvey.com>
Parts:
- C34, C35, C36: Field10 (none) -> Multilayer Ceramic; Field11 (none) -> other,more,stuff; Field4 (none) -> newark,39K8137; Field5 (none) -> vendor1, smd w hem; Field6 (none) -> vendor2, thru w hem; Field7 (none) -> vendor2, smd w hem; Field8 (none) -> 50,V; Field9 (none) -> 10,%
- D49, D50, D51, D52, D53, D54: Field10 (none) -> x; Field11 (none) -> other,more,stuff; Field4 (none) -> newark,10M2940; Field5 (none) -> vendor1, smd w hem; Field6 (none) -> vendor2, thru w hem; Field7 (none) -> vendor2, smd w hem; Field8 (none) -> 1000,V; Field9 (none) -> 1,A
- R64, R65, R66: value 1k -> 470R; TOL (none) -> 5%; W (none) -> 1/4W; construct (none) -> carbon film; misc (none) -> other,more,stuff; vend1,smd e hem (none) -> newark,42K4556; vend2, smd w hem (none) -> digi,CRCW0805470RFKEA; vend2, thru w hem (none) -> digi,CW02B470R0JE70-ND; vendor1, thru e hem (none) -> newark,65K3814
- R68, R69, R70: value 1k -> 0R; TOL (none) -> 5%; W (none) -> 1/4W; construct (none) -> carbon film; misc (none) -> other,more,stuff; vend1,smd e hem (none) -> newark,36C9353; vend2, smd w hem (none) -> digi,CRCW08050000ZSTA-ND; vend2, thru w hem (none) -> digi,604HR025E-ND; vendor1, thru e hem (none) -> newark,64K9335
