File: freeEMS_1.sch (KiCad schematic (older format))
At the start: 11 parts, among them P1 CONN_1, P2 CONN_1, P3 CONN_1, P4 CONN_1, P5 CONN_1, U1 74HC86, U2 74HC86

Commit message: DFH mans up a bit. Perhaps usable for something at this point, like making trips to the local store ;)
I connected TA pins to sub circuits, fixed a number if items discussed in the DIYEFI forums. This is it's 21st version, so it was time for it to man up a bit, and become something potentially useful.

Signed-off-by: Jared Harvey <TortiseGIT@jaredharvey.com>
Parts:
- added P101: CONN_1, 1PIN, symbol CONN_1
- added P102, P103, P104, P105, P106, P107: CONN_1, SIL-1, symbol CONN_1
- F1, F2, F3: Field10 (none) -> construct; Field11 (none) -> other,more,stuff; Field4 (none) -> newark,63K6823; Field5 (none) -> vendor1, smd w hem; Field6 (none) -> vendor2, thru w hem; Field7 (none) -> vendor2, smd w hem; Field8 (none) -> x,x; Field9 (none) -> 10,A
- RP1: Field4 (none) -> newark,32K8448
- U1, U2: Field10 (none) -> x; Field11 (none) -> x,x,x; Field4 (none) -> newark, 06F3172; Field5 (none) -> vendor1, smd w hem; Field6 (none) -> vendor2, thru e hem; Field7 (none) -> vendor2, smd e hem; Field8 (none) -> x,x; Field9 (none) -> x,x
Connections:
- net CPU/PT2 is gone; now on net ind_pd_1: RP1.14 (R3)
- net CPU/PT3 is gone; now on net ind_pd_2: RP1.13 (R4)
- net CPU/PT4 is gone; now on net ind_pd_3: RP1.12 (R5)
- net CPU/PT5 is gone; now on net ind_pd_4: RP1.11 (R6)
- net CPU/PT6 is gone; now on net ind_pd_5: RP1.10 (R7)
- net CPU/PT7 is gone; now on net ind_pd_6: RP1.9 (R8)
- net VCC_CNST: now also P101.1
- net ind_dr_1: now also U1.6 (OUT2); no longer U1.3 (OUT1)
- net ind_dr_2: now also U1.3 (OUT1); no longer U1.6 (OUT2)
- net ind_dr_3: now also U2.8 (OUT3); no longer U2.3 (OUT1)
- net ind_dr_5: now also U2.11 (OUT4); no longer U2.8 (OUT3)
- net ind_dr_6: now also U2.3 (OUT1); no longer U2.11 (OUT4)
- net ind_pd_1: now also P107.1
- net ind_pd_2: now also P106.1
- net ind_pd_3: now also P105.1
- net ind_pd_4: now also P104.1
- net ind_pd_5: now also P103.1
- net ind_pd_6: now also P102.1
- no-connect marks 65 -> 77
Other:
- note added: "JUMPER WIRE TO TA BOARD"
- note added: "jumper select if you want ignition, or fuel channels. Currently supports 6 channels total."
- moved on the sheet: RP1
