File: injector_drive5.sch (KiCad schematic (older format))
At the start: 17 parts, among them P34 CONN_1, P35 CONN_1, Q18 PIP-3104, Q19 HALL

Commit message: DFH mans up a bit. Perhaps usable for something at this point, like making trips to the local store ;)
I connected TA pins to sub circuits, fixed a number if items discussed in the DIYEFI forums. This is it's 21st version, so it was time for it to man up a bit, and become something potentially useful.

Signed-off-by: Jared Harvey <TortiseGIT@jaredharvey.com>
Parts:
- removed D93: ZENER 4V7, D4-SMB, symbol ZENER
- removed L5: INDUCTOR, SIL-2, symbol INDUCTOR
- removed Q19: HALL, SIL-3, symbol HALL
- removed R132: 0R, R4-SM0805, symbol R
- removed R133: 2.2k, R4-SM0805, symbol R
- removed R134: 680R, R4-SM0805, symbol R
- C53: Field10 (none) -> Multilayer Ceramic; Field11 (none) -> other,more,stuff; Field4 (none) -> newark,97M4148; Field5 (none) -> vendor1, smd w hem; Field6 (none) -> vendor2, thru w hem; Field7 (none) -> vendor2, smd w hem; Field8 (none) -> 200,V; Field9 (none) -> 10,%
- D92, D95: Field10 (none) -> x; Field11 (none) -> other,more,stuff; Field4 (none) -> vendor1, thru w hem; Field5 (none) -> vendor1, smd w hem; Field6 (none) -> vendor2, thru w hem; Field7 (none) -> vendor2, smd w hem; Field8 (none) -> reverse,V; Field9 (none) -> current,A
- D94: A (none) -> 10mA; V (none) -> 12V; construct (none) -> LED with resistor included; misc (none) -> other,more,stuff; vend1,smd e hem (none) -> newark,; vend2, smd w hem (none) -> digi,; vend2, thru w hem (none) -> digi,; vendor1, thru e hem (none) -> newark,58K2517
- Q18: value PIP-3104 -> MOSFET; A (none) -> 28A; V (none) -> 42V; construct (none) -> OVP protected MOSFET; misc (none) -> other,more,stuff; vend1,smd e hem (none) -> newark,; vend2, smd w hem (none) -> digi,; vend2, thru w hem (none) -> digi,VNP28N04-E-ND; vendor1, thru e hem (none) -> element14,1739427
- R129: W (none) -> 1/4w; construct (none) -> carbon film; misc (none) -> other,more,stuff; tol (none) -> 5%; vend1,smd e hem (none) -> newark,52K9725; vend2, smd w hem (none) -> digi,CRCW08051K00JNEA; vend2, thru w hem (none) -> digi,OD102J-ND; vendor1, thru e hem (none) -> newark,65K2365
- R130: Field10 (none) -> carbon film; Field11 (none) -> other,more,stuff; Field4 (none) -> newark,38K0329; Field5 (none) -> vendor1, smd w hem; Field6 (none) -> vendor2, thru w hem; Field7 (none) -> vendor2, smd w hem; Field8 (none) -> 250,mW; Field9 (none) -> 5,%
- R131: Field10 (none) -> carbon film; Field11 (none) -> other,more,stuff; Field4 (none) -> newark,38k0352; Field5 (none) -> vendor1, smd w hem; Field6 (none) -> vendor2, thru w hem; Field7 (none) -> vendor2, smd w hem; Field8 (none) -> 250,mW; Field9 (none) -> 5,%
- R135: value 3k -> 1k; W (none) -> 1/4w; construct (none) -> carbon film; misc (none) -> other,more,stuff; tol (none) -> 5%; vend1,smd e hem (none) -> newark,52K9725; vend2, smd w hem (none) -> digi,CRCW08051K00JNEA; vend2, thru w hem (none) -> digi,OD102J-ND; vendor1, thru e hem (none) -> newark,65K2365
Connections:
- net labels removed: current_sense
- wire segments 35 -> 21
Other:
- note removed: "CURRENT SENSE FEATURES"
- note removed: "CURRENT SENSING ALLOWS YOU TO MEASURE WHEN THE INJECTOR IS ON VS OFF"
