File: power_reg1.sch (KiCad schematic (older format))
At the start: 10 parts, among them U4 7805-DIYEFI

Commit message: DFH mans up a bit. Perhaps usable for something at this point, like making trips to the local store ;)
I connected TA pins to sub circuits, fixed a number if items discussed in the DIYEFI forums. This is it's 21st version, so it was time for it to man up a bit, and become something potentially useful.

Signed-off-by: Jared Harvey <TortiseGIT@jaredharvey.com>
Parts:
- C10: Field10 (none) -> Aluminum Electrolytic; Field11 (none) -> other,more,stuff; Field4 (none) -> newark,69K8230; Field5 (none) -> vendor1, smd w hem; Field6 (none) -> vendor2, thru w hem; Field7 (none) -> vendor2, smd w hem; Field8 (none) -> 50,V; Field9 (none) -> x,x
- C11, C8: Field10 (none) -> Tantalum; Field11 (none) -> other,more,stuff; Field4 (none) -> newark,97M4217; Field5 (none) -> vendor1, smd w hem; Field6 (none) -> vendor2, thru w hem; Field7 (none) -> vendor2, smd w hem; Field8 (none) -> 35,V; Field9 (none) -> 10,%
- C12, C9: Field10 (none) -> multilayer ceramic; Field11 (none) -> other,more,stuff; Field4 (none) -> newark,97M4164; Field5 (none) -> vendor1, smd w hem; Field6 (none) -> vendor2, thru w hem; Field7 (none) -> vendor2, smd w hem; Field8 (none) -> 50,V; Field9 (none) -> 20,%
- C7: Field10 (none) -> Aluminum Electrolytic; Field11 (none) -> other,more,stuff; Field4 (none) -> newark,69K8230; Field5 (none) -> vendor1, smd w hem; Field6 (none) -> vendor2, thru w hem; Field7 (none) -> vendor2, smd w hem; Field8 (none) -> 50,V; Field9 (none) -> X,%
- D11, D12: Field10 (none) -> construct; Field11 (none) -> other,more,stuff; Field4 (none) -> newark,18C8923; Field5 (none) -> DIGI,S1MBDIDKR-ND; Field6 (none) -> DIGI,1N4007RLOSCT-ND; Field7 (none) -> vendor2, smd w hem; Field8 (none) -> max,V; Field9 (none) -> x,x
- R10: Field10 (none) -> construct; Field11 (none) -> other,more,stuff; Field4 (none) -> newark, 65K3871; Field5 (none) -> farnell,1155286; Field6 (none) -> vendor2, thru w hem; Field7 (none) -> vendor2, smd w hem; Field8 (none) -> power,W; Field9 (none) -> tol,%
- U4: Field10 (none) -> linear; Field11 (none) -> other,more,stuff; Field4 (none) -> newark,45J1442; Field5 (none) -> vendor1, smd w hem; Field6 (none) -> vendor2, thru w hem; Field7 (none) -> vendor2, smd w hem; Field8 (none) -> x,x; Field9 (none) -> x,x
