File: thermistor_resistor_input1.sch (KiCad schematic (older format))
At the start: 4 parts, among them P53 CONN_1, P54 CONN_1, Q23 MOS_N

Commit message: DFH mans up a bit. Perhaps usable for something at this point, like making trips to the local store ;)
I connected TA pins to sub circuits, fixed a number if items discussed in the DIYEFI forums. This is it's 21st version, so it was time for it to man up a bit, and become something potentially useful.

Signed-off-by: Jared Harvey <TortiseGIT@jaredharvey.com>
Parts:
- Q23: Field10 (none) -> TOPFET; Field11 (none) -> other,more,stuff; Field4 (none) -> digi,PIP3104-ND; Field5 (none) -> vendor1, smd w hem; Field6 (none) -> vendor2, thru w hem; Field7 (none) -> vendor2, smd w hem; Field8 (none) -> 8,A; Field9 (none) -> x,x
- R178: Field10 (none) -> metal film; Field11 (none) -> other,more,stuff; Field4 (none) -> newark,41K8850; Field5 (none) -> vendor1, smd w hem; Field6 (none) -> vendor2, thru w hem; Field7 (none) -> vendor2, smd w hem; Field8 (none) -> .125,W; Field9 (none) -> 1,%
Changed lines of the file:
@@
-EESchema Schematic File Version 1
-LIBS:power,./freeEMS_lib,device,conn,linear,regul,74xx,cmos4000,adc-dac,memory,xilinx,special,microcontrollers,dsp,microchip,analog_switches,motorola,texas,intel,audio,interface,digital-audio,philips,display,cypress,siliconi,contrib,valves,./freeEMS_1.cache
-EELAYER 23  0
+EESchema Schematic File Version 2  date 9/10/2011 11:43:52 AM
+LIBS:power
+LIBS:freeEMS_lib
+LIBS:device
+LIBS:conn
+LIBS:linear
+LIBS:regul
+LIBS:74xx
+LIBS:cmos4000
+LIBS:adc-dac
+LIBS:memory
+LIBS:xilinx
+LIBS:special
+LIBS:microcontrollers
+LIBS:dsp
+LIBS:microchip
+LIBS:analog_switches
+LIBS:motorola
+LIBS:texas
+LIBS:intel
+LIBS:audio
+LIBS:interface
+LIBS:digital-audio
+LIBS:philips
+LIBS:display
+LIBS:cypress
+LIBS:siliconi
+LIBS:contrib
+LIBS:valves
+LIBS:freeEMS_1-cache
+EELAYER 25  0
 EELAYER END
 $Descr A 11000 8500
+encoding utf-8
 Sheet 40 41
-Title "freeEMS 1.0"
-Date "15 nov 2008"
-Rev "A.20"
-Comp "diyefi.org"
+Title "DFH for freeEMS"
+Date "10 sep 2011"
+Rev "A.21"
+Comp "FreeEMS.org"
 Comment1 "thermistor_resistor_input.sch"
 Comment2 ""
@@
 $Comp
 L PIP-3104 Q23
-U 1 1 48B16ED5
+U 1 1 4E6B7076
 P 3200 2150
-F 0 "Q23" H 3210 2320 60  0000 R C
-F 1 "MOS_N" H 3210 2000 60  0000 R C
-F 2 "TO92" V 3130 2900 60  0001 C C
-F 4 "digi,PIP3104-ND" V 1330 3900 60  0001 C C
-F 5 "vendor1, smd w hem" V 1330 3900 60  0001 C C
-F 6 "vendor2, thru w hem" V 1330 3900 60  0001 C C
-F 7 "vendor2, smd w hem" V 1330 3900 60  0001 C C
-F 8 "8,A" V 1330 3900 60  0001 C C
-F 9 "x,x" V 1330 3900 60  0001 C C
-F 10 "TOPFET" V 1330 3900 60  0001 C C
-F 11 "other,more,stuff" V 1330 3900 60  0001 C C
+F 0 "Q23" H 3210 2320 60  0000 R CNN
+F 1 "MOS_N" H 3210 2000 60  0000 R CNN
+F 2 "TO92" V 3130 2900 60  0001 C CNN
+F 4 "digi,PIP3104-ND" V 1330 3900 60  0001 C CNN "Field4"
+F 5 "vendor1, smd w hem" V 1330 3900 60  0001 C CNN "Field5"
+F 6 "vendor2, thru w hem" V 1330 3900 60  0001 C CNN "Field6"
+F 7 "vendor2, smd w hem" V 1330 3900 60  0001 C CNN "Field7"
+F 8 "8,A" V 1330 3900 60  0001 C CNN "Field8"
+F 9 "x,x" V 1330 3900 60  0001 C CNN "Field9"
+F 10 "TOPFET" V 1330 3900 60  0001 C CNN "Field10"
+F 11 "other,more,stuff" V 1330 3900 60  0001 C CNN "Field11"
 	1    3200 2150
 	1    0    0    -1
@@
 $Comp
 L CONN_1 P54
-U 1 1 48AA1AB3
+U 1 1 4E6B7047
 P 3450 1950
-F 0 "P54" H 3530 1950 40  0000 L C
-F 1 "CONN_1" H 3450 2005 30  0001 C C
-F 2 "1PIN" V 1130 2600 60  0001 C C
+F 0 "P54" H 3530 1950 40  0000 L CNN
+F 1 "CONN_1" H 3450 2005 30  0001 C CNN
+F 2 "1PIN" V 1130 2600 60  0001 C CNN
 	1    3450 1950
 	1    0    0    -1
@@
 $Comp
 L CONN_1 P53
-U 1 1 48AA1AB0
+U 1 1 4E6B7046
 P 3450 1750
-F 0 "P53" H 3530 1750 40  0000 L C
-F 1 "CONN_1" H 3450 1805 30  0001 C C
-F 2 "1PIN" V 1130 2600 60  0001 C C
+F 0 "P53" H 3530 1750 40  0000 L CNN
+F 1 "CONN_1" H 3450 1805 30  0001 C CNN
+F 2 "1PIN" V 1130 2600 60  0001 C CNN
 	1    3450 1750
 	1    0    0    -1
 $EndComp
-Text GLabel 2700 950  0    60   Output
+Text HLabel 2700 950  0    60   Output ~ 0
 5v_reg
 $Comp
 L R R178
-U 1 1 488E4A25
+U 1 1 4E6B6FED
 P 3300 1200
-F 0 "R178" V 3380 1200 50  0000 C C
-F 1 "2.7k" V 3300 1200 50  0000 C C
-F 2 "R4-SM0805" V 3480 1300 60  0001 C C
-F 4 "newark,41K8850" V 1130 2600 60  0001 C C
-F 5 "vendor1, smd w hem" V 1130 2600 60  0001 C C
-F 6 "vendor2, thru w hem" V 1130 2600 60  0001 C C
-F 7 "vendor2, smd w hem" V 1130 2600 60  0001 C C
-F 8 ".125,W" V 1130 2600 60  0001 C C
-F 9 "1,%" V 1130 2600 60  0001 C C
-F 10 "metal film" V 1130 2600 60  0001 C C
-F 11 "other,more,stuff" V 1130 2600 60  0001 C C
+F 0 "R178" V 3380 1200 50  0000 C CNN
+F 1 "2.7k" V 3300 1200 50  0000 C CNN
+F 2 "R4-SM0805" V 3480 1300 60  0001 C CNN
+F 4 "newark,41K8850" V 1130 2600 60  0001 C CNN "Field4"
+F 5 "vendor1, smd w hem" V 1130 2600 60  0001 C CNN "Field5"
+F 6 "vendor2, thru w hem" V 1130 2600 60  0001 C CNN "Field6"
+F 7 "vendor2, smd w hem" V 1130 2600 60  0001 C CNN "Field7"
+F 8 ".125,W" V 1130 2600 60  0001 C CNN "Field8"
+F 9 "1,%" V 1130 2600 60  0001 C CNN "Field9"
+F 10 "metal film" V 1130 2600 60  0001 C CNN "Field10"
+F 11 "other,more,stuff" V 1130 2600 60  0001 C CNN "Field11"
 	1    3300 1200
 	1    0    0    -1
 $EndComp
-Text GLabel 2650 2150 0    60   Input
+Text HLabel 2650 2150 0    60   Input ~ 0
 Measure_temp
-Text GLabel 2650 2350 0    60   BiDi
+Text HLabel 2650 2350 0    60   BiDi ~ 0
 analog_sensor_gnd
-Text GLabel 2700 1450 0    60   Output
+Text HLabel 2700 1450 0    60   Output ~ 0
 analog_sensor_TEMP
 $EndSCHEMATC
